File: Bioreactor/Bioreactor.sch (KiCad schematic (older format))
At the start: 11 parts, among them J1 Conn_01x03, J2 Conn_01x03, U1 ESP32-DEVKITC-32D, U2 MAX31855KASA

Commit message: ESP32 schematic recreation
Parts:
- removed J1, J2, J?: Conn_01x03, symbol Connector_Generic:Conn_01x03
- removed J?: Conn_01x02, symbol Connector_Generic:Conn_01x02
- removed J?: Barrel_Jack, symbol Connector:Barrel_Jack
- removed J?: Conn_01x04, symbol Connector_Generic:Conn_01x04
- removed R? (x2): R, symbol Device:R
- removed U1: ESP32-DEVKITC-32D, MODULE_ESP32-DEVKITC-32D, symbol ESP32-DEVKITC-32D:ESP32-DEVKITC-32D
- removed U2: MAX31855KASA, Package_SO:SOIC-8_3.9x4.9mm_P1.27mm, symbol Sensor_Temperature:MAX31855KASA
- removed U?: R-785.0-1.0, Converter_DCDC:Converter_DCDC_RECOM_R-78E-0.5_THT, symbol Regulator_Switching:R-785.0-1.0
- added J1: Jack-DC, symbol Connector:Jack-DC
- added J? (x2): Conn_01x03, symbol Connector_Generic:Conn_01x03
- added J?: Conn_01x04, symbol Connector_Generic:Conn_01x04
- added J? (x3): Conn_Coaxial, symbol Connector:Conn_Coaxial
- added R? (x2): 4.7K, symbol Device:R
- added U1: ESP32-DEVKITC-V1, MODULE_ESP32-DEVKITC-32D, symbol ESP32:ESP32-DEVKITC-V1
- added U2: LM7824_TO220, Package_TO_SOT_THT:TO-220-3_Vertical, symbol Regulator_Linear:LM7824_TO220
- added U?: MAX31855KASA, Package_SO:SOIC-8_3.9x4.9mm_P1.27mm, symbol Sensor_Temperature:MAX31855KASA
Connections:
- net labels added: +24V, +3V3, AMPLITUDE, MISO, MOSI, PHASE, SCK, TRIGGER, _CS
- net labels removed: VCC
- wire segments 52 -> 62
- no-connect marks 2 -> 16
